Commit message: Somewhat promising

File: src/jump_start/urdf/custom_turtlebot_gazebo.urdf.xacro (robot description, xacro)
@@ -40,6 +40,7 @@
     </gazebo>
   </xacro:macro> -->
-  <gazebo reference="camera_link1">
-     <sensor type="camera" name="camera1">
+<xacro:macro name="turtlebot_sim_3dsensor">
+ <gazebo reference="oleft">
+     <sensor type="camera" name="camera_left">
        <update_rate>30.0</update_rate>
         <camera name="head">
@@ -64,11 +65,10 @@
         </camera>
        <plugin name="camera_controller" filename="libgazebo_ros_camera.so">
-         <cameraName>camera1</cameraName>
+         <cameraName>left</cameraName>
          <alwaysOn>true</alwaysOn>
          <updateRate>0.0</updateRate>
-         <cameraName>camera1</cameraName>
          <imageTopicName>image_raw</imageTopicName>
-         <cameraInfoTopicName>camera1_info</cameraInfoTopicName>
-         <frameName>camera1_link</frameName>
+         <cameraInfoTopicName>camera_info</cameraInfoTopicName>
+         <frameName>left</frameName>
          <hackBaseline>0.07</hackBaseline>
          <distortionK1>0.0</distortionK1>
@@ -80,6 +80,6 @@
      </sensor>
    </gazebo>
- <gazebo reference="camera_link2">
-   <sensor type="camera" name="camera2">
+ <gazebo reference="right">
+   <sensor type="camera" name="camera_right">
      <update_rate>30.0</update_rate>
       <camera name="head">
@@ -104,11 +104,10 @@
       </camera>
      <plugin name="camera_controller" filename="libgazebo_ros_camera.so">
-       <cameraName>camera2</cameraName>
+       <cameraName>right</cameraName>
        <alwaysOn>true</alwaysOn>
        <updateRate>0.0</updateRate>
-       <cameraName>camera2</cameraName>
        <imageTopicName>image_raw</imageTopicName>
-       <cameraInfoTopicName>camera2_info</cameraInfoTopicName>
-       <frameName>camera2_link</frameName>
+       <cameraInfoTopicName>camera_info</cameraInfoTopicName>
+       <frameName>right</frameName>
        <hackBaseline>0.07</hackBaseline>
        <distortionK1>0.0</distortionK1>
@@ -120,3 +119,4 @@
    </sensor>
  </gazebo>
+</xacro:macro>
 </robot>

File: src/jump_start/urdf/sensors/custom.urdf.xacro (robot description, xacro)
@@ -22,7 +22,7 @@
       <origin xyz="0.15 ${custom_cam_py} -0.016" rpy="0 0 0"/>
       <parent link="camera_rgb_frame"/>
-      <child link="camera_link1"/>
+      <child link="oleft"/>
     </joint>
-      <link name="camera_link1">
+      <link name="oleft">
       <visual>
        <origin xyz="0 0 0" rpy="0 0 ${M_PI/2}"/>
@@ -49,7 +49,7 @@
       <origin xyz="0.15 ${-custom_cam_py} -0.016" rpy="0 0 0"/>
       <parent link="camera_rgb_frame"/>
-      <child link="camera_link2"/>
+      <child link="right"/>
     </joint>
-      <link name="camera_link2">
+      <link name="right">
       <visual>
        <origin xyz="0 0 0" rpy="0 0 ${M_PI/2}"/>
@@ -73,9 +73,15 @@
       </inertial>
     </link>
+    <joint name="camera_joint3" type="fixed">
+      <origin xyz="0.15 ${custom_cam_py} -0.016" rpy="-${M_PI/2} 0 -${M_PI/2}"/>
+      <parent link="camera_rgb_frame"/>
+      <child link="left"/>
+    </joint>
+      <link name="left" />
     <!-- The fixed joints & links below are usually published by static_transformers launched by the OpenNi launch
          files. However, for Gazebo simulation we need them, so we add them here.
          (Hence, don't publish them additionally!) -->
-	<!-- Kinect sensor for simulation -->
-	<!-- <turtlebot_sim_3dsensor/> -->
+	<!-- Custom sensor for simulation -->
+	<turtlebot_sim_3dsensor/>
   </xacro:macro>
 </robot>

File: src/jump_start/urdf/sensors/kinect.urdf.xacro (robot description, xacro)
@@ -3,10 +3,9 @@
   <xacro:include filename="$(find turtlebot_description)/urdf/turtlebot_gazebo.urdf.xacro"/>
   <xacro:include filename="$(find turtlebot_description)/urdf/turtlebot_properties.urdf.xacro"/>
-  <xacro:property name="camera_link" value="0.035" /> <!-- Size of square 'camera' box -->
-  <xacro:property name="kinect_cam_py" value="0.075"/>
+  <xacro:property name="kinect_cam_py" value="-0.0125"/>
   <!-- Parameterised in part by the values in turtlebot_properties.urdf.xacro -->
   <xacro:macro name="sensor_kinect" params="parent">
     <joint name="camera_rgb_joint" type="fixed">
-      <origin xyz="${cam_px} 0 ${cam_pz}" rpy="${cam_or} ${cam_op} ${cam_oy}"/>
+      <origin xyz="${cam_px} ${kinect_cam_py} ${cam_pz}" rpy="${cam_or} ${cam_op} ${cam_oy}"/>
       <parent link="${parent}"/>
       <child link="camera_rgb_frame" />
@@ -19,43 +18,15 @@
     </joint>
     <link name="camera_rgb_optical_frame"/>
-    <joint name="camera_joint1" type="fixed">
-      <origin xyz="0.15 ${kinect_cam_py} -0.016" rpy="0 0 0"/>
+    <joint name="camera_joint" type="fixed">
+      <origin xyz="-0.031 ${-kinect_cam_py} -0.016" rpy="0 0 0"/>
       <parent link="camera_rgb_frame"/>
-      <child link="camera_link1"/>
+      <child link="camera_link"/>
     </joint>
-      <link name="camera_link1">
+      <link name="camera_link">
       <visual>
        <origin xyz="0 0 0" rpy="0 0 ${M_PI/2}"/>
-       <geometry>
-         <box size="${camera_link} ${camera_link} ${camera_link}"/>
-         <material name="red"/>
-       </geometry>
-      </visual>
-  	  <collision>
-        <origin xyz="0.0 0.0 0.0" rpy="0 0 0"/>
-  	    <geometry>
-  	      <box size="0.07271 0.27794 0.073"/>
-  	    </geometry>
-  	  </collision>
-      <inertial>
-        <mass value="0.564" />
-        <origin xyz="0 0 0" />
-        <inertia ixx="0.003881243" ixy="0.0" ixz="0.0"
-                 iyy="0.000498940" iyz="0.0"
-                 izz="0.003879257" />
-      </inertial>
-    </link>
-    <joint name="camera_joint2" type="fixed">
-      <origin xyz="0.15 ${-kinect_cam_py} -0.016" rpy="0 0 0"/>
-      <parent link="camera_rgb_frame"/>
-      <child link="camera_link2"/>
-    </joint>
-      <link name="camera_link2">
-      <visual>
-       <origin xyz="0 0 0" rpy="0 0 ${M_PI/2}"/>
-       <geometry>
-         <box size="${camera_link} ${camera_link} ${camera_link}"/>
-         <material name="red"/>
-       </geometry>
+        <geometry>
+         <mesh filename="package://turtlebot_description/meshes/sensors/kinect.dae"/>
+        </geometry>
       </visual>
   	  <collision>
@@ -76,6 +47,18 @@
          files. However, for Gazebo simulation we need them, so we add them here.
          (Hence, don't publish them additionally!) -->
+	<joint name="camera_depth_joint" type="fixed">
+	  <origin xyz="0 ${2 * -kinect_cam_py} 0" rpy="0 0 0" />
+	  <parent link="camera_rgb_frame" />
+	  <child link="camera_depth_frame" />
+	</joint>
+	<link name="camera_depth_frame"/>
+	<joint name="camera_depth_optical_joint" type="fixed">
+	  <origin xyz="0 0 0" rpy="${-M_PI/2} 0 ${-M_PI/2}" />
+	  <parent link="camera_depth_frame" />
+	  <child link="camera_depth_optical_frame" />
+	</joint>
+	<link name="camera_depth_optical_frame"/>
 	<!-- Kinect sensor for simulation -->
-	<!-- <turtlebot_sim_3dsensor/> -->
+	<xacro:turtlebot_sim_3dsensor/>
   </xacro:macro>
 </robot>

Commit message: rtabmap is working

File: src/jump_start/urdf/custom_turtlebot_gazebo.urdf.xacro (robot description, xacro)
@@ -41,47 +41,8 @@
   </xacro:macro> -->
 <xacro:macro name="turtlebot_sim_3dsensor">
- <gazebo reference="oleft">
-     <sensor type="camera" name="camera_left">
-       <update_rate>30.0</update_rate>
-        <camera name="head">
-          <horizontal_fov>1.3962634</horizontal_fov>
-          <image>
-            <width>800</width>
-            <height>800</height>
-            <format>R8G8B8</format>
-          </image>
-          <clip>
-            <near>0.02</near>
-            <far>300</far>
-          </clip>
-          <noise>
-            <type>gaussian</type>
-            <!-- Noise is sampled independently per pixel on each frame.
-                 That pixel's noise value is added to each of its color
-                 channels, which at that point lie in the range [0,1]. -->
-            <mean>0.0</mean>
-            <stddev>0.007</stddev>
-          </noise>
-        </camera>
-       <plugin name="camera_controller" filename="libgazebo_ros_camera.so">
-         <cameraName>left</cameraName>
-         <alwaysOn>true</alwaysOn>
-         <updateRate>0.0</updateRate>
-         <imageTopicName>image_raw</imageTopicName>
-         <cameraInfoTopicName>camera_info</cameraInfoTopicName>
-         <frameName>left</frameName>
-         <hackBaseline>0.07</hackBaseline>
-         <distortionK1>0.0</distortionK1>
-         <distortionK2>0.0</distortionK2>
-         <distortionK3>0.0</distortionK3>
-         <distortionT1>0.0</distortionT1>
-         <distortionT2>0.0</distortionT2>
-       </plugin>
-     </sensor>
-   </gazebo>
- <gazebo reference="right">
-   <sensor type="camera" name="camera_right">
-     <update_rate>30.0</update_rate>
-      <camera name="head">
+<gazebo reference="oleft">
+    <sensor type="multicamera" name="stereo_camera">
+      <update_rate>30.0</update_rate>
+      <camera name="left">
         <horizontal_fov>1.3962634</horizontal_fov>
         <image>
@@ -96,27 +57,43 @@
         <noise>
           <type>gaussian</type>
-          <!-- Noise is sampled independently per pixel on each frame.
-               That pixel's noise value is added to each of its color
-               channels, which at that point lie in the range [0,1]. -->
           <mean>0.0</mean>
           <stddev>0.007</stddev>
         </noise>
       </camera>
-     <plugin name="camera_controller" filename="libgazebo_ros_camera.so">
-       <cameraName>right</cameraName>
-       <alwaysOn>true</alwaysOn>
-       <updateRate>0.0</updateRate>
-       <imageTopicName>image_raw</imageTopicName>
-       <cameraInfoTopicName>camera_info</cameraInfoTopicName>
-       <frameName>right</frameName>
-       <hackBaseline>0.07</hackBaseline>
-       <distortionK1>0.0</distortionK1>
-       <distortionK2>0.0</distortionK2>
-       <distortionK3>0.0</distortionK3>
-       <distortionT1>0.0</distortionT1>
-       <distortionT2>0.0</distortionT2>
-     </plugin>
-   </sensor>
- </gazebo>
-</xacro:macro>
+      <camera name="right">
+        <pose>0 -0.07 0 0 0 0</pose>
+        <horizontal_fov>1.3962634</horizontal_fov>
+        <image>
+          <width>800</width>
+          <height>800</height>
+          <format>R8G8B8</format>
+        </image>
+        <clip>
+          <near>0.02</near>
+          <far>300</far>
+        </clip>
+        <noise>
+          <type>gaussian</type>
+          <mean>0.0</mean>
+          <stddev>0.007</stddev>
+        </noise>
+      </camera>
+      <plugin name="stereo_camera_controller" filename="libgazebo_ros_multicamera.so">
+        <alwaysOn>true</alwaysOn>
+        <updateRate>0.0</updateRate>
+        <cameraName>stereo/camera</cameraName>
+        <imageTopicName>image_raw</imageTopicName>
+        <cameraInfoTopicName>camera_info</cameraInfoTopicName>
+        <frameName>left</frameName>
+        <!--<rightFrameName>right_camera_optical_frame</rightFrameName>-->
+        <hackBaseline>0.07</hackBaseline>
+        <distortionK1>0.0</distortionK1>
+        <distortionK2>0.0</distortionK2>
+        <distortionK3>0.0</distortionK3>
+        <distortionT1>0.0</distortionT1>
+        <distortionT2>0.0</distortionT2>
+      </plugin>
+    </sensor>
+  </gazebo>
+  </xacro:macro>
 </robot>

Commit message: Finally something works, don't know why

File: src/jump_start/urdf/custom_turtlebot_gazebo.urdf.xacro (robot description, xacro)
@@ -82,5 +82,5 @@
         <alwaysOn>true</alwaysOn>
         <updateRate>0.0</updateRate>
-        <cameraName>stereo/camera</cameraName>
+        <cameraName>stereo</cameraName>
         <imageTopicName>image_raw</imageTopicName>
         <cameraInfoTopicName>camera_info</cameraInfoTopicName>

File: src/jump_start/urdf/sensors/custom.urdf.xacro (robot description, xacro)
@@ -20,9 +20,9 @@
     <link name="camera_rgb_optical_frame"/>
     <joint name="camera_joint1" type="fixed">
-      <origin xyz="0.15 ${custom_cam_py} -0.016" rpy="0 0 0"/>
+      <origin xyz="0.15 ${custom_cam_py} -0.016" rpy="${-M_PI/2} 0 ${-M_PI/2}"/>
       <parent link="camera_rgb_frame"/>
-      <child link="oleft"/>
+      <child link="left"/>
     </joint>
-      <link name="oleft">
+      <link name="left">
       <visual>
        <origin xyz="0 0 0" rpy="0 0 ${M_PI/2}"/>
@@ -74,9 +74,9 @@
     </link>
     <joint name="camera_joint3" type="fixed">
-      <origin xyz="0.15 ${custom_cam_py} -0.016" rpy="-${M_PI/2} 0 -${M_PI/2}"/>
+      <origin xyz="0.15 ${custom_cam_py} -0.016" rpy="0 0 0"/>
       <parent link="camera_rgb_frame"/>
-      <child link="left"/>
+      <child link="oleft"/>
     </joint>
-      <link name="left" />
+      <link name="oleft" />
     <!-- The fixed joints & links below are usually published by static_transformers launched by the OpenNi launch
          files. However, for Gazebo simulation we need them, so we add them here.
